File: Circuit/Hall_sensor_array/Hall_sensor_array.kicad_pcb (KiCad board)
At the start: 2 copper layers, 768 parts, among them U1 AH49HSC, U10 AH49HSC, U100 AH49HSC, U101 AH49HSC, U102 AH49HSC, U103 AH49HSC, U104 AH49HSC, U105 AH49HSC, U106 AH49HSC, U107 AH49HSC, U108 AH49HSC, U109 AH49HSC, U11 AH49HSC, U110 AH49HSC, U111 AH49HSC, U112 AH49HSC, U113 AH49HSC, U114 AH49HSC, U115 AH49HSC, U116 AH49HSC, U117 AH49HSC, U118 AH49HSC, U119 AH49HSC, U12 AH49HSC, U120 AH49HSC, U121 AH49HSC, U122 AH49HSC, U123 AH49HSC, U124 AH49HSC, U125 AH49HSC, U126 AH49HSC, U127 AH49HSC, U128 AH49HSC, U129 AH49HSC, U13 AH49HSC, U130 AH49HSC, U131 AH49HSC, U132 AH49HSC, U133 AH49HSC, U134 AH49HSC, U135 AH49HSC, U136 AH49HSC, U137 AH49HSC, U138 AH49HSC, U139 AH49HSC, U14 AH49HSC, U140 AH49HSC, U141 AH49HSC, U142 AH49HSC, U143 AH49HSC, U144 AH49HSC, U145 AH49HSC, U146 AH49HSC, U147 AH49HSC, U148 AH49HSC, U149 AH49HSC, U15 AH49HSC, U150 AH49HSC, U151 AH49HSC, U152 AH49HSC, U153 AH49HSC, U154 AH49HSC, U155 AH49HSC, U156 AH49HSC, U157 AH49HSC, U158 AH49HSC, U159 AH49HSC, U16 AH49HSC, U160 AH49HSC, U161 AH49HSC, U162 AH49HSC, U163 AH49HSC, U164 AH49HSC, U165 AH49HSC, U166 AH49HSC, U167 AH49HSC, U168 AH49HSC, U169 AH49HSC, U17 AH49HSC, U170 AH49HSC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

Commit message: Updated circuit(work in progress)
Parts:
- removed C257, C258, C259, C260, C261, C262, C263, C264, C265, C266, C267, C268, C269, C270, C271, C272, C289, C290, C291, C292, C293, C294, C295, C296, C297, C298, C299, C300, C301, C302, C303, C304, C321, C322, C323, C324, C325, C326, C327, C328, C329, C330, C331, C332, C333, C334, C335, C336, C353, C354, C355, C356, C357, C358, C359, C360, C361, C362, C363, C364, C365, C366, C367, C368, C385, C386, C387, C388, C389, C390, C391, C392, C393, C394, C395, C396, C397, C398, C399, C400, C417, C418, C419, C420, C421, C422, C423, C424, C425, C426, C427, C428, C429, C430, C431, C432, C449, C450, C451, C452, C453, C454, C455, C456, C457, C458, C459, C460, C461, C462, C463, C464, C481, C482, C483, C484, C485, C486, C487, C488, C489, C490, C491, C492, C493, C494, C495: 10n, Capacitor_SMD:C_0603_1608Metric
- removed C273, C274, C275, C276, C277, C278, C279, C280, C281, C282, C283, C284, C285, C286, C287, C288, C305, C306, C307, C308, C309, C310, C311, C312, C313, C314, C315, C316, C317, C318, C319, C320, C337, C338, C339, C340, C341, C342, C343, C344, C345, C346, C347, C348, C349, C350, C351, C352, C369, C370, C371, C372, C373, C374, C375, C376, C377, C378, C379, C380, C381, C382, C383, C384, C401, C402, C403, C404, C405, C406, C407, C408, C409, C410, C411, C412, C413, C414, C415, C416, C433, C434, C435, C436, C437, C438, C439, C440, C441, C442, C443, C444, C445, C446, C447, C448, C465, C466, C467, C468, C469, C470, C471, C472, C473, C474, C475, C476, C477, C478, C479, C480, C497, C498, C499, C500, C501, C502, C503, C504, C505, C506, C507, C508, C509, C510, C511, C512: 100p, Capacitor_SMD:C_0603_1608Metric
- added U257: CD74HC4067SM, Package_SO:TSSOP-24_4.4x7.8mm_P0.65mm, B.Cu at (-327.8, -88.2)
- added U258: CD74HC4067SM, Package_SO:TSSOP-24_4.4x7.8mm_P0.65mm, F.Cu at (171.6, 55.7)
- added U259: CD74HC4067SM, Package_SO:TSSOP-24_4.4x7.8mm_P0.65mm, F.Cu at (136.6, 65.0)
- added U260: CD74HC4067SM, Package_SO:TSSOP-24_4.4x7.8mm_P0.65mm, F.Cu at (180.3, 55.7)
- added U261: CD74HC4067SM, Package_SO:TSSOP-24_4.4x7.8mm_P0.65mm, F.Cu at (154.1, 55.7)
- added U262: CD74HC4067SM, Package_SO:TSSOP-24_4.4x7.8mm_P0.65mm, F.Cu at (162.8, 74.4)
- added U263: CD74HC4067SM, Package_SO:TSSOP-24_4.4x7.8mm_P0.65mm, F.Cu at (162.8, 65.0)
- added U264: CD74HC4067SM, Package_SO:TSSOP-24_4.4x7.8mm_P0.65mm, F.Cu at (162.8, 55.7)
- added U265: CD74HC4067SM, Package_SO:TSSOP-24_4.4x7.8mm_P0.65mm, F.Cu at (136.6, 55.7)
- added U266: CD74HC4067SM, Package_SO:TSSOP-24_4.4x7.8mm_P0.65mm, F.Cu at (145.3, 74.4)
- added U267: CD74HC4067SM, Package_SO:TSSOP-24_4.4x7.8mm_P0.65mm, F.Cu at (154.1, 74.4)
- added U268: CD74HC4067SM, Package_SO:TSSOP-24_4.4x7.8mm_P0.65mm, F.Cu at (171.6, 65.0)
- added U269: CD74HC4067SM, Package_SO:TSSOP-24_4.4x7.8mm_P0.65mm, F.Cu at (145.3, 65.0)
- added U270: CD74HC4067SM, Package_SO:TSSOP-24_4.4x7.8mm_P0.65mm, F.Cu at (136.6, 74.4)
- added U271: CD74HC4067SM, Package_SO:TSSOP-24_4.4x7.8mm_P0.65mm, F.Cu at (154.1, 65.0)
- added U272: CD74HC4067SM, Package_SO:TSSOP-24_4.4x7.8mm_P0.65mm, F.Cu at (145.3, 55.7)
- added U273: ESP32-WROVER-IE-N8R8, RF_Module:ESP32-WROVER-IE-N8R8, F.Cu at (74.8, 86.3)
- added U274: ADS7830, Package_SO:TSSOP-16_4.4x5mm_P0.65mm, F.Cu at (55.5, 113.8)
- C1, C10, C100, C101, C102, C103, C104, C105, C106, C107, C108, C109, C11, C110, C111, C112, C12, C129, C13, C130, C131, C132, C133, C134, C135, C136, C137, C138, C139, C14, C140, C141, C142, C143, C144, C15, C16, C161, C162, C163, C164, C165, C166, C167, C168, C169, C170, C171, C172, C173, C174, C175, C176, C193, C194, C195, C196, C197, C198, C199, C2, C200, C201, C202, C203, C204, C205, C206, C207, C208, C225, C226, C227, C228, C229, C230, C231, C232, C233, C234, C235, C236, C237, C238, C239, C240, C3, C33, C34, C35, C36, C37, C38, C39, C4, C40, C41, C42, C43, C44, C45, C46, C47, C48, C5, C6, C65, C66, C67, C68, C69, C7, C70, C71, C72, C73, C74, C75, C76, C77, C78, C79, C8, C80, C9, C97, C98, C99: value 10n -> 100p
- moved C496 533.3 mm to (93.0, 127.4)
- moved C1 516.9 mm to (-337.4, -78.2), turned to -90 degrees
- moved C10 516.9 mm to (-337.4, 56.8), turned to -90 degrees
- moved C11 516.9 mm to (-337.4, 71.8), turned to -90 degrees
- moved C12 516.9 mm to (-337.4, 86.8), turned to -90 degrees
- moved C13 516.9 mm to (-337.4, 101.8), turned to -90 degrees
- moved C14 516.9 mm to (-337.4, 116.8), turned to -90 degrees
- moved C15 516.9 mm to (-337.4, 131.8), turned to -90 degrees
- moved C16 516.9 mm to (-337.4, 146.8), turned to -90 degrees
- moved C2 516.9 mm to (-337.4, -63.2), turned to -90 degrees
- moved C3 516.9 mm to (-337.4, -48.2), turned to -90 degrees
- moved C4 516.9 mm to (-337.4, -33.2), turned to -90 degrees
- moved C5 516.9 mm to (-337.4, -18.2), turned to -90 degrees
- moved C6 516.9 mm to (-337.4, -3.16), turned to -90 degrees
- moved C7 516.9 mm to (-337.4, 11.8), turned to -90 degrees
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Connections:
- C1 pad 1: +3.3V -> X1Y1
- C10 pad 1: +3.3V -> X1Y10
- C100 pad 1: +3.3V -> X7Y4
- C101 pad 1: +3.3V -> X7Y5
- C102 pad 1: +3.3V -> X7Y6
- C103 pad 1: +3.3V -> X7Y7
- C104 pad 1: +3.3V -> X7Y8
- C105 pad 1: +3.3V -> X7Y9
- C106 pad 1: +3.3V -> X7Y10
- C107 pad 1: +3.3V -> X7Y11
- C108 pad 1: +3.3V -> X7Y12
- C109 pad 1: +3.3V -> X7Y13
- C11 pad 1: +3.3V -> X1Y11
- C110 pad 1: +3.3V -> X7Y14
- C111 pad 1: +3.3V -> X7Y15
- C112 pad 1: +3.3V -> X7Y16
- C113 pad 1: X4Y1 -> X8Y1
- C114 pad 1: X4Y2 -> X8Y2
- C115 pad 1: X4Y3 -> X8Y3
- C116 pad 1: X4Y4 -> X8Y4
- C117 pad 1: X4Y5 -> X8Y5
- C118 pad 1: X4Y6 -> X8Y6
- C119 pad 1: X4Y7 -> X8Y7
- C12 pad 1: +3.3V -> X1Y12
- C120 pad 1: X4Y8 -> X8Y8
- C121 pad 1: X4Y9 -> X8Y9
- C122 pad 1: X4Y10 -> X8Y10
- C123 pad 1: X4Y11 -> X8Y11
- C124 pad 1: X4Y12 -> X8Y12
- C125 pad 1: X4Y13 -> X8Y13
- C126 pad 1: X4Y14 -> X8Y14
- C127 pad 1: X4Y15 -> X8Y15
- C128 pad 1: X4Y16 -> X8Y16
- C129 pad 1: +3.3V -> X9Y1
- C13 pad 1: +3.3V -> X1Y13
- C130 pad 1: +3.3V -> X9Y2
- C131 pad 1: +3.3V -> X9Y3
- C132 pad 1: +3.3V -> X9Y4
- C133 pad 1: +3.3V -> X9Y5
- C134 pad 1: +3.3V -> X9Y6
- C135 pad 1: +3.3V -> X9Y7
- C136 pad 1: +3.3V -> X9Y8
- C137 pad 1: +3.3V -> X9Y9
- C138 pad 1: +3.3V -> X9Y10
- C139 pad 1: +3.3V -> X9Y11
- C14 pad 1: +3.3V -> X1Y14
- C140 pad 1: +3.3V -> X9Y12
- C141 pad 1: +3.3V -> X9Y13
- C142 pad 1: +3.3V -> X9Y14
- C143 pad 1: +3.3V -> X9Y15
- C144 pad 1: +3.3V -> X9Y16
- C145 pad 1: X5Y1 -> X10Y1
- C146 pad 1: X5Y2 -> X10Y2
- C147 pad 1: X5Y3 -> X10Y3
- C148 pad 1: X5Y4 -> X10Y4
- C149 pad 1: X5Y5 -> X10Y5
- C15 pad 1: +3.3V -> X1Y15
- C150 pad 1: X5Y6 -> X10Y6
- C151 pad 1: X5Y7 -> X10Y7
- C152 pad 1: X5Y8 -> X10Y8
- C153 pad 1: X5Y9 -> X10Y9
- C154 pad 1: X5Y10 -> X10Y10
- C155 pad 1: X5Y11 -> X10Y11
- C156 pad 1: X5Y12 -> X10Y12
- C157 pad 1: X5Y13 -> X10Y13
- C158 pad 1: X5Y14 -> X10Y14
- C159 pad 1: X5Y15 -> X10Y15
- C16 pad 1: +3.3V -> X1Y16
- C160 pad 1: X5Y16 -> X10Y16
- C161 pad 1: +3.3V -> X11Y1
- C162 pad 1: +3.3V -> X11Y2
- C163 pad 1: +3.3V -> X11Y3
- C164 pad 1: +3.3V -> X11Y4
- C165 pad 1: +3.3V -> X11Y5
- C166 pad 1: +3.3V -> X11Y6
- C167 pad 1: +3.3V -> X11Y7
- C168 pad 1: +3.3V -> X11Y8
- C169 pad 1: +3.3V -> X11Y9
- C17 pad 1: X1Y1 -> X2Y1
- C170 pad 1: +3.3V -> X11Y10
- C171 pad 1: +3.3V -> X11Y11
- C172 pad 1: +3.3V -> X11Y12
- C173 pad 1: +3.3V -> X11Y13
- C174 pad 1: +3.3V -> X11Y14
- C175 pad 1: +3.3V -> X11Y15
- C176 pad 1: +3.3V -> X11Y16
- C177 pad 1: X6Y1 -> X12Y1
- C178 pad 1: X6Y2 -> X12Y2
- C179 pad 1: X6Y3 -> X12Y3
- C18 pad 1: X1Y2 -> X2Y2
- C180 pad 1: X6Y4 -> X12Y4
- C181 pad 1: X6Y5 -> X12Y5
- C182 pad 1: X6Y6 -> X12Y6
- C183 pad 1: X6Y7 -> X12Y7
- C184 pad 1: X6Y8 -> X12Y8
- C185 pad 1: X6Y9 -> X12Y9
- C186 pad 1: X6Y10 -> X12Y10
- C187 pad 1: X6Y11 -> X12Y11
- C188 pad 1: X6Y12 -> X12Y12
- C189 pad 1: X6Y13 -> X12Y13
- C19 pad 1: X1Y3 -> X2Y3
- C190 pad 1: X6Y14 -> X12Y14
- C191 pad 1: X6Y15 -> X12Y15
- C192 pad 1: X6Y16 -> X12Y16
- C193 pad 1: +3.3V -> X13Y1
- C194 pad 1: +3.3V -> X13Y2
- C195 pad 1: +3.3V -> X13Y3
- C196 pad 1: +3.3V -> X13Y4
- C197 pad 1: +3.3V -> X13Y5
- C198 pad 1: +3.3V -> X13Y6
- C199 pad 1: +3.3V -> X13Y7
- C2 pad 1: +3.3V -> X1Y2
- C20 pad 1: X1Y4 -> X2Y4
- C200 pad 1: +3.3V -> X13Y8
- C201 pad 1: +3.3V -> X13Y9
- C202 pad 1: +3.3V -> X13Y10
- C203 pad 1: +3.3V -> X13Y11
- C204 pad 1: +3.3V -> X13Y12
- C205 pad 1: +3.3V -> X13Y13
- C206 pad 1: +3.3V -> X13Y14
- C207 pad 1: +3.3V -> X13Y15
- C208 pad 1: +3.3V -> X13Y16
- C209 pad 1: X7Y1 -> X14Y1
- C21 pad 1: X1Y5 -> X2Y5
- C210 pad 1: X7Y2 -> X14Y2
- C211 pad 1: X7Y3 -> X14Y3
- C212 pad 1: X7Y4 -> X14Y4
- C213 pad 1: X7Y5 -> X14Y5
- C214 pad 1: X7Y6 -> X14Y6
- C215 pad 1: X7Y7 -> X14Y7
- C216 pad 1: X7Y8 -> X14Y8
- C217 pad 1: X7Y9 -> X14Y9
- C218 pad 1: X7Y10 -> X14Y10
- C219 pad 1: X7Y11 -> X14Y11
- C22 pad 1: X1Y6 -> X2Y6
- C220 pad 1: X7Y12 -> X14Y12
- C221 pad 1: X7Y13 -> X14Y13
- C222 pad 1: X7Y14 -> X14Y14
- C223 pad 1: X7Y15 -> X14Y15
- C224 pad 1: X7Y16 -> X14Y16
- C225 pad 1: +3.3V -> X15Y1
- C226 pad 1: +3.3V -> X15Y2
- C227 pad 1: +3.3V -> X15Y3
- C228 pad 1: +3.3V -> X15Y4
- C229 pad 1: +3.3V -> X15Y5
- C23 pad 1: X1Y7 -> X2Y7
- C230 pad 1: +3.3V -> X15Y6
- C231 pad 1: +3.3V -> X15Y7
- C232 pad 1: +3.3V -> X15Y8
- C233 pad 1: +3.3V -> X15Y9
- C234 pad 1: +3.3V -> X15Y10
- C235 pad 1: +3.3V -> X15Y11
- C236 pad 1: +3.3V -> X15Y12
- C237 pad 1: +3.3V -> X15Y13
- C238 pad 1: +3.3V -> X15Y14
- C239 pad 1: +3.3V -> X15Y15
- C24 pad 1: X1Y8 -> X2Y8
- C240 pad 1: +3.3V -> X15Y16
- C241 pad 1: X8Y1 -> X16Y1
- C242 pad 1: X8Y2 -> X16Y2
- C243 pad 1: X8Y3 -> X16Y3
- C244 pad 1: X8Y4 -> X16Y4
- C245 pad 1: X8Y5 -> X16Y5
- C246 pad 1: X8Y6 -> X16Y6
- C247 pad 1: X8Y7 -> X16Y7
- C248 pad 1: X8Y8 -> X16Y8
- C249 pad 1: X8Y9 -> X16Y9
- C25 pad 1: X1Y9 -> X2Y9
- C250 pad 1: X8Y10 -> X16Y10
- C251 pad 1: X8Y11 -> X16Y11
- C252 pad 1: X8Y12 -> X16Y12
- C253 pad 1: X8Y13 -> X16Y13
- C254 pad 1: X8Y14 -> X16Y14
- C255 pad 1: X8Y15 -> X16Y15
- C256 pad 1: X8Y16 -> X16Y16
- C26 pad 1: X1Y10 -> X2Y10
- C27 pad 1: X1Y11 -> X2Y11
- C28 pad 1: X1Y12 -> X2Y12
- C29 pad 1: X1Y13 -> X2Y13
- C3 pad 1: +3.3V -> X1Y3
- C30 pad 1: X1Y14 -> X2Y14
- C31 pad 1: X1Y15 -> X2Y15
- C32 pad 1: X1Y16 -> X2Y16
- C33 pad 1: +3.3V -> X3Y1
- C34 pad 1: +3.3V -> X3Y2
- C35 pad 1: +3.3V -> X3Y3
- C36 pad 1: +3.3V -> X3Y4
- C37 pad 1: +3.3V -> X3Y5
- C38 pad 1: +3.3V -> X3Y6
- C39 pad 1: +3.3V -> X3Y7
- C4 pad 1: +3.3V -> X1Y4
- C40 pad 1: +3.3V -> X3Y8
- C41 pad 1: +3.3V -> X3Y9
- C42 pad 1: +3.3V -> X3Y10
- C43 pad 1: +3.3V -> X3Y11
- C44 pad 1: +3.3V -> X3Y12
- C45 pad 1: +3.3V -> X3Y13
- C46 pad 1: +3.3V -> X3Y14
- C47 pad 1: +3.3V -> X3Y15
- C48 pad 1: +3.3V -> X3Y16
- C49 pad 1: X2Y1 -> X4Y1
- C496 pad 1: +3.3V -> (no net)
- C496 pad 2: GND -> (no net)
- C5 pad 1: +3.3V -> X1Y5
- C50 pad 1: X2Y2 -> X4Y2
- C51 pad 1: X2Y3 -> X4Y3
- C52 pad 1: X2Y4 -> X4Y4
- C53 pad 1: X2Y5 -> X4Y5
- C54 pad 1: X2Y6 -> X4Y6
- C55 pad 1: X2Y7 -> X4Y7
- C56 pad 1: X2Y8 -> X4Y8
- C57 pad 1: X2Y9 -> X4Y9
- C58 pad 1: X2Y10 -> X4Y10
- C59 pad 1: X2Y11 -> X4Y11
- C6 pad 1: +3.3V -> X1Y6
- C60 pad 1: X2Y12 -> X4Y12
- C61 pad 1: X2Y13 -> X4Y13
- C62 pad 1: X2Y14 -> X4Y14
- C63 pad 1: X2Y15 -> X4Y15
- C64 pad 1: X2Y16 -> X4Y16
- C65 pad 1: +3.3V -> X5Y1
- C66 pad 1: +3.3V -> X5Y2
- C67 pad 1: +3.3V -> X5Y3
- C68 pad 1: +3.3V -> X5Y4
- C69 pad 1: +3.3V -> X5Y5
- C7 pad 1: +3.3V -> X1Y7
- C70 pad 1: +3.3V -> X5Y6
- C71 pad 1: +3.3V -> X5Y7
- C72 pad 1: +3.3V -> X5Y8
- C73 pad 1: +3.3V -> X5Y9
- C74 pad 1: +3.3V -> X5Y10
- C75 pad 1: +3.3V -> X5Y11
- C76 pad 1: +3.3V -> X5Y12
- C77 pad 1: +3.3V -> X5Y13
- C78 pad 1: +3.3V -> X5Y14
- C79 pad 1: +3.3V -> X5Y15
- C8 pad 1: +3.3V -> X1Y8
- C80 pad 1: +3.3V -> X5Y16
- C81 pad 1: X3Y1 -> X6Y1
- C82 pad 1: X3Y2 -> X6Y2
- C83 pad 1: X3Y3 -> X6Y3
- C84 pad 1: X3Y4 -> X6Y4
- C85 pad 1: X3Y5 -> X6Y5
- C86 pad 1: X3Y6 -> X6Y6
- C87 pad 1: X3Y7 -> X6Y7
- C88 pad 1: X3Y8 -> X6Y8
- C89 pad 1: X3Y9 -> X6Y9
- C9 pad 1: +3.3V -> X1Y9
- C90 pad 1: X3Y10 -> X6Y10
- C91 pad 1: X3Y11 -> X6Y11
- C92 pad 1: X3Y12 -> X6Y12
- C93 pad 1: X3Y13 -> X6Y13
- C94 pad 1: X3Y14 -> X6Y14
- C95 pad 1: X3Y15 -> X6Y15
- C96 pad 1: X3Y16 -> X6Y16
- C97 pad 1: +3.3V -> X7Y1
- C98 pad 1: +3.3V -> X7Y2
- C99 pad 1: +3.3V -> X7Y3
Routing:
- net X1Y16: track 0.00 -> 245.6 mm, vias 0 -> 1
- net X1Y15: track 0.00 -> 230.0 mm, vias 0 -> 1
- net X1Y14: track 0.00 -> 214.3 mm, vias 0 -> 1
- net GND: track 0.00 -> 211.4 mm, vias 0 -> 256
- net X1Y13: track 0.00 -> 198.7 mm, vias 0 -> 1
- net X1Y12: track 0.00 -> 183.1 mm, vias 0 -> 1
- net X1Y11: track 0.00 -> 167.5 mm, vias 0 -> 1
- net X1Y10: track 0.00 -> 151.9 mm, vias 0 -> 1
- net X1Y9: track 0.00 -> 136.2 mm, vias 0 -> 1
- net X1Y8: track 0.00 -> 129.9 mm, vias 0 -> 1
- net X1Y7: track 0.00 -> 116.2 mm, vias 0 -> 1
- net X1Y6: track 0.00 -> 102.8 mm, vias 0 -> 1
- net X1Y5: track 0.00 -> 89.3 mm, vias 0 -> 1
- net X1Y4: track 0.00 -> 75.8 mm, vias 0 -> 1
- net X1Y3: track 0.00 -> 62.2 mm, vias 0 -> 1
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