File: Circuit/Hall_sensor_array/Analog_multiplexing.kicad_sch (KiCad schematic)
At the start: 32 parts, among them U257 CD74HC4067SM, U258 CD74HC4067SM, U259 CD74HC4067SM, U260 CD74HC4067SM, U261 CD74HC4067SM, U262 CD74HC4067SM, U263 CD74HC4067SM, U264 CD74HC4067SM, U265 CD74HC4067SM, U266 CD74HC4067SM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

Commit message: Updated circuit
Added binary counter for selecting analog multiplexer address
Parts:
- added R17: 1k, symbol Device:R
- added U276: CD74HC4067SM, Package_SO:TSSOP-24_4.4x7.8mm_P0.65mm, symbol 74xx:CD74HC4067SM
Connections:
- net +9V: now also U276.24 (VCC)
- net E: now also R17.1
- net GND: now also U276.12 (GND)
- net X1: now also U276.9 (I0)
- net X10: now also U276.22 (I9)
- net X11: now also U276.21 (I10)
- net X12: now also U276.20 (I11)
- net X13: now also U276.19 (I12)
- net X14: now also U276.18 (I13)
- net X15: now also U276.17 (I14)
- net X16: now also U276.16 (I15)
- net X2: now also U276.8 (I1)
- net X3: now also U276.7 (I2)
- net X4: now also U276.6 (I3)
- net X5: now also U276.5 (I4)
- net X6: now also U276.4 (I5)
- net X7: now also U276.3 (I6)
- net X8: now also U276.2 (I7)
- net X9: now also U276.23 (I8)
- net X16Y16: now reaches U262.16 (I15)
- net X16Y15: now reaches U262.17 (I14)
- net X16Y14: now reaches U262.18 (I13)
- new net: R17.2, U276.15 (~{E})
- new net A_out: U276.1 (COM)
- new net S4: U276.10 (S0)
- new net S5: U276.11 (S1)
- new net S6: U276.14 (S2)
- new net S7: U276.13 (S3)
