File: Circuit/Hall_sensor_array/Hall_sensor_array.kicad_sch (KiCad schematic)
At the start: 768 parts, among them U1 AH49HSC, U10 AH49HSC, U100 AH49HSC, U101 AH49HSC, U102 AH49HSC, U103 AH49HSC, U104 AH49HSC, U105 AH49HSC, U106 AH49HSC, U107 AH49HSC, U108 AH49HSC, U109 AH49HSC, U11 AH49HSC, U110 AH49HSC, U111 AH49HSC, U112 AH49HSC, U113 AH49HSC, U114 AH49HSC, U115 AH49HSC, U116 AH49HSC, U117 AH49HSC, U118 AH49HSC, U119 AH49HSC, U12 AH49HSC, U120 AH49HSC, U121 AH49HSC, U122 AH49HSC, U123 AH49HSC, U124 AH49HSC, U125 AH49HSC, U126 AH49HSC, U127 AH49HSC, U128 AH49HSC, U129 AH49HSC, U13 AH49HSC, U130 AH49HSC, U131 AH49HSC, U132 AH49HSC, U133 AH49HSC, U134 AH49HSC, U135 AH49HSC, U136 AH49HSC, U137 AH49HSC, U138 AH49HSC, U139 AH49HSC, U14 AH49HSC, U140 AH49HSC, U141 AH49HSC, U142 AH49HSC, U143 AH49HSC, U144 AH49HSC, U145 AH49HSC, U146 AH49HSC, U147 AH49HSC, U148 AH49HSC, U149 AH49HSC, U15 AH49HSC, U150 AH49HSC, U151 AH49HSC, U152 AH49HSC, U153 AH49HSC, U154 AH49HSC, U155 AH49HSC, U156 AH49HSC, U157 AH49HSC, U158 AH49HSC, U159 AH49HSC, U16 AH49HSC, U160 AH49HSC, U161 AH49HSC, U162 AH49HSC, U163 AH49HSC, U164 AH49HSC, U165 AH49HSC, U166 AH49HSC, U167 AH49HSC, U168 AH49HSC, U169 AH49HSC, U17 AH49HSC, U170 AH49HSC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

Commit message: Updated circuit(work in progress)
Parts:
- removed C1, C10, C100, C101, C102, C103, C104, C105, C106, C107, C108, C109, C11, C110, C111, C112, C12, C129, C13, C130, C131, C132, C133, C134, C135, C136, C137, C138, C139, C14, C140, C141, C142, C143, C144, C15, C16, C161, C162, C163, C164, C165, C166, C167, C168, C169, C170, C171, C172, C173, C174, C175, C176, C193, C194, C195, C196, C197, C198, C199, C2, C200, C201, C202, C203, C204, C205, C206, C207, C208, C225, C226, C227, C228, C229, C230, C231, C232, C233, C234, C235, C236, C237, C238, C239, C240, C257, C258, C259, C260, C261, C262, C263, C264, C265, C266, C267, C268, C269, C270, C271, C272, C289, C290, C291, C292, C293, C294, C295, C296, C297, C298, C299, C3, C300, C301, C302, C303, C304, C321, C322, C323, C324, C325, C326, C327, C328, C329, C33, C330, C331, C332, C333, C334, C335, C336, C34, C35, C353, C354, C355, C356, C357, C358, C359, C36, C360, C361, C362, C363, C364, C365, C366, C367, C368, C37, C38, C385, C386, C387, C388, C389, C39, C390, C391, C392, C393, C394, C395, C396, C397, C398, C399, C4, C40, C400, C41, C417, C418, C419, C42, C420, C421, C422, C423, C424, C425, C426, C427, C428, C429, C43, C430, C431, C432, C44, C449, C45, C450, C451, C452, C453, C454, C455, C456, C457, C458, C459, C46, C460, C461, C462, C463, C464, C47, C48, C481, C482, C483, C484, C485, C486, C487, C488, C489, C490, C491, C492, C493, C494, C495, C496, C5, C6, C65, C66, C67, C68, C69, C7, C70, C71, C72, C73, C74, C75, C76, C77, C78, C79, C8, C80, C9, C97, C98, C99: 10n, Capacitor_SMD:C_0603_1608Metric, symbol Device:C
- removed C113, C114, C115, C116, C117, C118, C119, C120, C121, C122, C123, C124, C125, C126, C127, C128, C145, C146, C147, C148, C149, C150, C151, C152, C153, C154, C155, C156, C157, C158, C159, C160, C17, C177, C178, C179, C18, C180, C181, C182, C183, C184, C185, C186, C187, C188, C189, C19, C190, C191, C192, C20, C209, C21, C210, C211, C212, C213, C214, C215, C216, C217, C218, C219, C22, C220, C221, C222, C223, C224, C23, C24, C241, C242, C243, C244, C245, C246, C247, C248, C249, C25, C250, C251, C252, C253, C254, C255, C256, C26, C27, C273, C274, C275, C276, C277, C278, C279, C28, C280, C281, C282, C283, C284, C285, C286, C287, C288, C29, C30, C305, C306, C307, C308, C309, C31, C310, C311, C312, C313, C314, C315, C316, C317, C318, C319, C32, C320, C337, C338, C339, C340, C341, C342, C343, C344, C345, C346, C347, C348, C349, C350, C351, C352, C369, C370, C371, C372, C373, C374, C375, C376, C377, C378, C379, C380, C381, C382, C383, C384, C401, C402, C403, C404, C405, C406, C407, C408, C409, C410, C411, C412, C413, C414, C415, C416, C433, C434, C435, C436, C437, C438, C439, C440, C441, C442, C443, C444, C445, C446, C447, C448, C465, C466, C467, C468, C469, C470, C471, C472, C473, C474, C475, C476, C477, C478, C479, C480, C49, C497, C498, C499, C50, C500, C501, C502, C503, C504, C505, C506, C507, C508, C509, C51, C510, C511, C512, C52, C53, C54, C55, C56, C57, C58, C59, C60, C61, C62, C63, C64, C81, C82, C83, C84, C85, C86, C87, C88, C89, C90, C91, C92, C93, C94, C95, C96: 100p, Capacitor_SMD:C_0603_1608Metric, symbol Device:C
- removed U1, U10, U100, U101, U102, U103, U104, U105, U106, U107, U108, U109, U11, U110, U111, U112, U113, U114, U115, U116, U117, U118, U119, U12, U120, U121, U122, U123, U124, U125, U126, U127, U128, U129, U13, U130, U131, U132, U133, U134, U135, U136, U137, U138, U139, U14, U140, U141, U142, U143, U144, U145, U146, U147, U148, U149, U15, U150, U151, U152, U153, U154, U155, U156, U157, U158, U159, U16, U160, U161, U162, U163, U164, U165, U166, U167, U168, U169, U17, U170, U171, U172, U173, U174, U175, U176, U177, U178, U179, U18, U180, U181, U182, U183, U184, U185, U186, U187, U188, U189, U19, U190, U191, U192, U193, U194, U195, U196, U197, U198, U199, U2, U20, U200, U201, U202, U203, U204, U205, U206, U207, U208, U209, U21, U210, U211, U212, U213, U214, U215, U216, U217, U218, U219, U22, U220, U221, U222, U223, U224, U225, U226, U227, U228, U229, U23, U230, U231, U232, U233, U234, U235, U236, U237, U238, U239, U24, U240, U241, U242, U243, U244, U245, U246, U247, U248, U249, U25, U250, U251, U252, U253, U254, U255, U256, U26, U27, U28, U29, U3, U30, U31, U32, U33, U34, U35, U36, U37, U38, U39, U4, U40, U41, U42, U43, U44, U45, U46, U47, U48, U49, U5, U50, U51, U52, U53, U54, U55, U56, U57, U58, U59, U6, U60, U61, U62, U63, U64, U65, U66, U67, U68, U69, U7, U70, U71, U72, U73, U74, U75, U76, U77, U78, U79, U8, U80, U81, U82, U83, U84, U85, U86, U87, U88, U89, U9, U90, U91, U92, U93, U94, U95, U96, U97, U98, U99: AH49HSC, Package_TO_SOT_SMD:SOT-23-3, symbol Sensor_Magnetic:AH49HSC
Other:
- added sheet ADC (ADC.kicad_sch)
- added sheet Analog_multiplexing (Analog_multiplexing.kicad_sch)
- added sheet Digital_electronics (Digital_electronics.kicad_sch)
- added sheet Power_filtering (Power_filtering.kicad_sch)
- added sheet Sensor_array (Sensor_array.kicad_sch)
