File: Circuit/Hall_sensor_array/Power_filtering.kicad_sch (KiCad schematic)
At the start: 9 parts, among them U273 ZD1117ILTR50, U274 78D06LL-TN3-R, U275 UZ1085L-33-TN3-R

Commit message: Major update! New pcb
i did some work
Parts:
- added C301, C302, C303, C304, C305, C306, C307, C308, C309, C310, C311, C312, C313, C314, C315, C316, C317: 100n, Capacitor_SMD:C_0603_1608Metric, symbol Device:C
- U273: footprint Package_TO_SOT_SMD:SOT-223 -> Package_TO_SOT_SMD:TO-252-2
- U275: value UZ1085L-33-TN3-R -> AZ1117D-3.3
Connections:
- net +6V: now also U274.3 (VO), C301.1, C302.1, C303.1, C304.1, C305.1, C306.1, C307.1, C308.1, C309.1, C310.1, C311.1, C312.1, C313.1, C314.1, C315.1, C316.1, C317.1; no longer U274.2 (VO)
- net GND: now also U274.2 (GND), C301.2, C302.2, C303.2, C304.2, C305.2, C306.2, C307.2, C308.2, C309.2, C310.2, C311.2, C312.2, C313.2, C314.2, C315.2, C316.2, C317.2; no longer U274.1 (GND)
- net VCC: now also U274.1 (VI); no longer U274.3 (VI)
Other:
- moved on the sheet: U274
